Commit message: IMPORTANT FIXES (aerial landing)

File: aerial_robot/robots/neo11_base.xacro (robot description, xacro)
@@ -18,4 +18,7 @@
 <robot name="neo11" xmlns:xacro="http://ros.org/wiki/xacro">
   <xacro:include filename="$(find rotors_description)/urdf/component_snippets.xacro" />
+  <xacro:arg name="namespace" default="neo11" />
+  <xacro:arg name="enable_ground_truth" default="false" />
+  <xacro:arg name="enable_logging" default="false" />
   <!-- Instantiate neo11 "mechanics" -->
   <xacro:include filename="$(find rotors_description)/urdf/neo11.xacro" />

File: commander/objects/beer.urdf (robot description, URDF)
Before this commit: robot beer, 1 links, 0 joints
Links:
- link world/beer_link: geometry collision box size=0.1 0.05 0.05; visual mesh filename=package://commander/meshes/beam.dae scale=0.2 0.2 0.2

File: commander/urdf/sphere_obstacle.urdf.xacro (robot description, xacro)
@@ -15,5 +15,5 @@
 				<origin xyz="${xyz}" />
 				<geometry>
-					<sphere radius="${r}" />
+					<mesh filename="package://commander/meshes/box.dae" scale="0.15 0.15 0.15"/>
 				</geometry>
 			</visual>
@@ -24,5 +24,5 @@
 		</link>
 		<gazebo reference="${name}">
-			<material>Gazebo/Blue</material>
+			<!--material>Gazebo/Blue</material-->
 			<static>true</static>
    			<turnGravityOff>true</turnGravityOff>

File: nexus_robot/urdf/nexus_base/base.urdf.xacro (robot description, xacro)
@@ -34,6 +34,6 @@
   <xacro:property name="wheel_joint_safety_k_velocity" value="100.0"/>
   <xacro:macro name="nexus_base" params="name">
-    <link name="${name}_footprint">
-      <collision>
+    <link name="${name}_footprint"
+>      <collision>
         <origin xyz="0 0 ${-base_size_z / 2.0}" rpy="0 0 0"/>
         <geometry>

File: nexus_robot/urdf/widowx_arm/widowx.urdf.xacro (robot description, xacro)
@@ -259,5 +259,5 @@
       </joint>
       <joint name="${prefix}gripper_prismatic_joint_1" type="fixed">
-         <origin xyz="0 -0.032 0" rpy="0 0 0" />
+         <origin xyz="0 -0.02 0" rpy="0 0 0" />
          <parent link="${prefix}gripper_rail_link" />
          <child link="${prefix}gripper_1_link" />
@@ -266,5 +266,5 @@
       </joint>
       <joint name="${prefix}gripper_prismatic_joint_2" type="fixed">
-         <origin xyz="0 0.032 0" rpy="0 0 0" />
+         <origin xyz="0 0.02 0" rpy="0 0 0" />
          <parent link="${prefix}gripper_rail_link" />
          <child link="${prefix}gripper_2_link" />
